Commit message: Fix LEDs pose and add light material

File: desistek_saga_description/urdf/desistek_saga_led.xacro (robot description, xacro)
@@ -6,5 +6,6 @@
     prefix="right"
     parent_link="${namespace}/base_link">
-    <origin xyz="0.2 -0.1192 0.0" rpy="0 0 0"/>
+    <origin xyz="0.1 -0.1192 0.0" rpy="0 0 0"/>
+    <pose xyz="0.1 -0.1192 0.0" rpy="0 0 0"/>
   </xacro:led_macro>
 <!-- Left LED -->
@@ -13,5 +14,6 @@
     parent_link="${namespace}/base_link"
     prefix="left">
-    <origin xyz="0.2 0.1192 0.0" rpy="0 0 0"/>
+    <origin xyz="0.1 0.1192 0.0" rpy="0 0 0"/>
+    <pose xyz="0.1 0.1192 0.0" rpy="0 0 0"/>
   </xacro:led_macro>
 </robot>

File: desistek_saga_description/urdf/desistek_saga_snippets.xacro (robot description, xacro)
@@ -27,11 +27,11 @@
   </xacro:macro>
   <xacro:macro name="led_macro"
-    params="namespace prefix parent_link *origin">
+    params="namespace prefix parent_link *origin *pose">
     <!-- LED link -->
     <link name="${namespace}/${prefix}_LED_link">
-      <!-- <light name='lamp' type='spot'>
-        <pose>0 0 0.0 0 3.14159 0</pose>
+      <light name='lamp' type='point'>
+        <pose>2 0 0.0 0 3.14159 0</pose>
         <attenuation>
-          <range>30</range>
+          <range>3</range>
           <linear>0.05</linear>
         </attenuation>
@@ -44,8 +44,8 @@
         </spot>
         <direction>0 0 -1</direction>
-      </light> -->
+      </light>
     <visual name='lamp_visual'>
       <geometry>
-        <sphere radius="0.005"/>
+        <sphere radius="0.02"/>
       </geometry>
     </visual>
@@ -69,5 +69,5 @@
       <!-- Understand if it is a relative or absolute position -->
       <!-- The light is carried with the robot, so, it should be relative -->
-        <pose>0 0 0 0 0 0</pose>
+        <xacro:insert_block name="pose" />
       </light>
       <plugin name='light_control' filename='libFlashLightPlugin.so'>
@@ -83,4 +83,7 @@
       <selfCollide>false</selfCollide>
     </gazebo>
+    <gazebo reference="${namespace}/${prefix}_LED_link">
+      <material>Gazebo/GreenGlow</material>
+    </gazebo>
   </xacro:macro>
 </robot>
